File: MegaDrive.kicad_pcb (KiCad board)
At the start: 2 copper layers, 239.3 x 191 mm, 291 parts, among them J1 Video, J10 Conn_01x04_Pin, J11 Conn_01x02_Pin, J110 Conn_01x04_Pin, J111 Conn_01x02_Socket, J2 Floppy, J3 Cartridge, J4 EXT, J5 Player1, J6 Player2, J7 Jack-DC, J8 AudioJack3, J9 Conn_01x02_Pin, J99 Conn_01x02_Pin, SW1 SW_SPDT, SW2 SW_Push, U1 HD68HC000P8, U10 M5M4C264L, U11 YM2612, U12 CXA1034P, U14 LM358, U15 L7805, U17 L7805, U2 uPD42832C-15, U3 uPD42832C-15, U4 315-5402, U6 Z80CPU, U7 uPD4364, U8 312-5313A, U9 M5M4C264L

Commit message: Add files via upload
Parts:
- removed RV1: 50K, SEGA:HeadphoneVolumeSlider
- removed U13: ~, Package_DIP:DIP-24_W10.16mm
- added C125: 100pF, MD1_VA6.8:C_0805_2012Metric, B.Cu at (87.8, 95.3)
- added IC13: MB3514, MD1_VA6.8:SOIC-24_CXA, F.Cu at (77.8, 94.2)
- added VR1: 50K, MD1_VA6.8:HeadphoneSlider, F.Cu at (40.5, 186.7)
- C1, C111, C13, C23, C24, C30, C31, C32, C38, C4, C40, C41, C42, C43, C44, C49, C5, C50, C51, C52, C53, C55, C57, C58, C59, C60, C61, C62, C63, C64, C65, C66, C68, C71, C72, C74, C79, C86, CP112: footprint Capacitor_THT:CP_Radial_Tantal_D4.5mm_P5.00mm -> MD1_VA6.8:CP_Radial_Tantal_D4.5mm_P5.00mm
- C10, C102, C103, C105, C106, C107, C108, C109, C11, C110, C112, C113, C114, C115, C116, C117, C118, C119, C120, C121, C122, C14, C15, C16, C17, C18, C19, C2, C20, C21, C22, C25, C26, C27, C28, C29, C3, C33, C34, C35, C37, C39, C45, C46, C47, C48, C6, C69, C7, C73, C75, C77, C78, C8, C80, C81, C82, C83, C85, C87, C88, C89, C9, C90, C91, C92, C93, C94, C95, C96: footprint Capacitor_SMD:C_0805_2012Metric -> MD1_VA6.8:C_0805_2012Metric
- CN1: renamed from J1; footprint SEGA:DIN8Video -> MD1_VA6.8:DIN8Video
- CN10: renamed from J10; footprint Connector_PinHeader_2.00mm:PinHeader_1x04_P2.00mm_Vertical -> MD1_VA6.8:PinHeader_1x04_P2.00mm_Vertical
- CN11: renamed from J11; footprint Connector_PinHeader_2.54mm:PinHeader_1x02_P2.54mm_Vertical -> MD1_VA6.8:PinHeader_1x02_P2.54mm_Vertical
- CN110: renamed from J110; footprint Connector_PinHeader_2.00mm:PinHeader_1x04_P2.00mm_Vertical -> MD1_VA6.8:PinHeader_1x04_P2.00mm_Vertical
- CN111: renamed from J111; footprint Connector_PinHeader_2.54mm:PinHeader_1x02_P2.54mm_Vertical -> MD1_VA6.8:PinHeader_1x02_P2.54mm_Vertical
- CN2: renamed from J2; footprint SEGA:Expansion -> MD1_VA6.8:Expansion
- CN3: renamed from J3; footprint SEGA:SEGA_2x32_Female_Vertical_THT -> MD1_VA6.8:SEGA_2x32_Female_Vertical_THT
- CN4: renamed from J4; footprint Connector_Dsub:DSUB-9_Socket_Horizontal_P2.77x2.84mm_EdgePinOffset9.40mm -> MD1_VA6.8:DSUB-9_Socket_Horizontal_P2.77x2.84mm_EdgePinOffset9.40mm
- CN5: renamed from J5; footprint Connector_Dsub:DSUB-9_Pins_Horizontal_P2.77x2.84mm_EdgePinOffset9.40mm -> MD1_VA6.8:DSUB-9_Pins_Horizontal_P2.77x2.84mm_EdgePinOffset9.40mm
- CN6: renamed from J6; footprint Connector_Dsub:DSUB-9_Pins_Horizontal_P2.77x2.84mm_EdgePinOffset9.40mm -> MD1_VA6.8:DSUB-9_Pins_Horizontal_P2.77x2.84mm_EdgePinOffset9.40mm
- CN7: renamed from J7; footprint SEGA:BarrelJack_CUI_PJ-002A_Horizontal -> MD1_VA6.8:BarrelJack_CUI_PJ-002A_Horizontal
- CN8: renamed from J8; footprint SEGA:Jack_3.5mm -> MD1_VA6.8:Jack_3.5mm
- CN9: renamed from J9; footprint Connector_PinSocket_2.54mm:PinSocket_1x02_P2.54mm_Vertical -> MD1_VA6.8:PinSocket_1x02_P2.54mm_Vertical
- CN99: renamed from J99; footprint Connector_PinSocket_2.54mm:PinSocket_1x02_P2.54mm_Vertical -> MD1_VA6.8:PinSocket_1x02_P2.54mm_Vertical
- D1, D2, D3: footprint Diode_THT:D_A-405_P5.08mm_Vertical_AnodeUp -> MD1_VA6.8:D_A-405_P5.08mm_Vertical_AnodeUp
- EM11, EM12, EM13, EM16, EM21, EM22, EM23, EM24, EM25, EM26, EM27, EM28, EM31, EM32, EM33, EM34, EM35, EM36, EM37, EM38, EM4, EM5, EM7, EM8: footprint Crystal:Resonator-3Pin_W6.0mm_H3.0mm -> MD1_VA6.8:Resonator-3Pin_W6.0mm_H3.0mm
- FB1, FB10, FB13, FB14, FB2, FB3, FB4, FB5, FB8, FB9, L6: footprint Inductor_THT:L_Axial_L7.0mm_D3.3mm_P5.08mm_Vertical_Fastron_MICC -> MD1_VA6.8:L_Axial_L7.0mm_D3.3mm_P5.08mm_Vertical_Fastron_MICC
- FB11, FB12, FB15, FB6, FB7: footprint Ferrite_THT:LairdTech_28C0236-0JW-10 -> MD1_VA6.8:LairdTech_28C0236-0JW-10
- FID1, FID2, FID3, FID4, FID5, FID6: footprint Fiducial:Fiducial_1.5mm_Mask4.5mm -> MD1_VA6.8:Fiducial_1.5mm_Mask4.5mm
- H1, H10, H11, H12, H2, H3, H4, H5, H7, H8, H9: footprint MountingHole:MountingHole_3.2mm_M3 -> MD1_VA6.8:MountingHole_3.2mm_M3
- H13, H14, H15: footprint MountingHole:MountingHole_5mm -> MD1_VA6.8:MountingHole_5mm
- H6: footprint MountingHole:MountingHole_4mm -> MD1_VA6.8:MountingHole_4mm
- IC1: renamed from U1; value HD68HC000P8 -> 68000P; footprint Package_DIP:DIP-64_W22.86mm -> MD1_VA6.8:DIP-64_W22.86mm
- IC10: renamed from U10; footprint SEGA:ZIP-24 -> MD1_VA6.8:ZIP-24
- IC11: renamed from U11; footprint Package_DIP:DIP-24_W15.24mm -> MD1_VA6.8:DIP-24_W15.24mm
- IC12: renamed from U12; footprint Package_DIP:DIP-16_W7.62mm -> MD1_VA6.8:DIP-16_W7.62mm
- IC14: renamed from U14; footprint Package_DIP:DIP-8_W7.62mm -> MD1_VA6.8:DIP-8_W7.62mm
- IC15: renamed from U15; footprint Package_TO_SOT_THT:TO-220-3_Vertical -> MD1_VA6.8:TO-220-3_Vertical
- IC17: renamed from U17; footprint Package_TO_SOT_THT:TO-220-3_Vertical -> MD1_VA6.8:TO-220-3_Vertical
- IC2: renamed from U2; footprint SEGA:DIP-28_DoubleLast -> MD1_VA6.8:DIP-28_DoubleLast
- IC3: renamed from U3; footprint SEGA:DIP-28_DoubleLast -> MD1_VA6.8:DIP-28_DoubleLast
- IC4: renamed from U4; value 315-5402 -> 315-5433; footprint SEGA:QFP-160_28x28_Pitch0.65mm -> MD1_VA6.8:QFP-160_28x28_Pitch0.65mm
- IC6: renamed from U6; footprint Package_DIP:DIP-40_W15.24mm -> MD1_VA6.8:DIP-40_W15.24mm
- IC7: renamed from U7; footprint SEGA:DIP-28_DoubleFirst -> MD1_VA6.8:DIP-28_DoubleFirst
- IC8: renamed from U8; value 312-5313A -> 315-5313A; footprint SEGA:QFP128 -> MD1_VA6.8:QFP128
- IC9: renamed from U9; footprint SEGA:ZIP-24 -> MD1_VA6.8:ZIP-24
- JP1, JP2, JP3, JP4, L2, L3, L5, L7: footprint Resistor_THT:R_Axial_DIN0204_L3.6mm_D1.6mm_P5.08mm_Horizontal -> MD1_VA6.8:R_Axial_DIN0204_L3.6mm_D1.6mm_P5.08mm_Horizontal
- JP5, JP6, JP7: footprint Connector_PinSocket_2.54mm:PinSocket_1x01_P2.54mm_Vertical -> MD1_VA6.8:PinSocket_1x01_P2.54mm_Vertical
- NT101: footprint NetTie:NetTie-2_SMD_Pad2.0mm -> MD1_VA6.8:NetTie-2_SMD_Pad2.0mm
- OSC1: footprint Oscillator:Oscillator_DIP-14 -> MD1_VA6.8:Oscillator_DIP-14
- R1, R10, R11, R12, R14, R15, R16, R17, R18, R19, R20, R21, R22, R23, R24, R25, R26, R29, R3, R30, R31, R32, R33, R34, R35, R36, R37, R38, R39, R4, R40, R41, R42, R43, R49, R5, R50, R51, R52, R53, R54, R55, R56, R57, R58, R59, R6, R64, R65, R66, R67, R68, R69, R7, R70, R71, R72, R73, R74, R77, R78, R79, R8, R80, R81, R82, R83, R84, R85, R9: footprint Resistor_SMD:R_0805_2012Metric -> MD1_VA6.8:R_0805_2012Metric
- R27: value 1.2k -> 560; footprint Resistor_SMD:R_0805_2012Metric -> MD1_VA6.8:R_0805_2012Metric
- R28: value 1.2k -> 3.3k; footprint Resistor_SMD:R_0805_2012Metric -> MD1_VA6.8:R_0805_2012Metric
- RF1: footprint SEGA:RFmod -> MD1_VA6.8:RFmod
- SW1: footprint Button_Switch_THT:SW_E-Switch_EG1224_SPDT_Angled -> MD1_VA6.8:SW_E-Switch_EG1224_SPDT_Angled
- SW2: footprint Button_Switch_THT:SW_Tactile_Straight_KSA0Axx1LFTR -> MD1_VA6.8:SW_Tactile_Straight_KSA0Axx1LFTR
- moved R28 16.7 mm to (75.5, 99.5), turned to 180 degrees
- moved R30 16.3 mm to (78.5, 83.2), turned to -90 degrees
- moved C95 10.4 mm to (81.0, 83.2), turned to 90 degrees
- moved R26 8.25 mm to (75.5, 102.0)
- moved C33 7.77 mm to (72.9, 95.3), turned to 90 degrees
- moved R29 7.39 mm to (73.5, 85.9), turned to -90 degrees
- moved R24 3.18 mm to (77.4, 109.7)
- moved R27 3.17 mm to (79.1, 88.8), turned to 90 degrees
- moved C38 3.09 mm to (70.7, 81.8), turned to 0 degrees
- moved C29 2.61 mm to (77.4, 106.6)
- moved C24 1.39 mm to (75.6, 76.0)
Routing:
- net GND: track 4714.1 -> 5074.8 mm, vias 128 -> 132
- net /~{RAS0}: track 41.5 -> 201.0 mm, vias 0 -> 4
- net VCC: track 899.1 -> 930.7 mm
- net VDDF: track 190.3 -> 217.6 mm, vias 2 -> 4
- net Net-(IC13-C_SYNC_IN): track 217.6 -> 243.6 mm, vias 3 -> 4
- net /VREF: track 83.3 -> 107.8 mm, vias 1 -> 2
- net Net-(C37-Pad1): track 43.2 -> 27.6 mm
- net Net-(IC13-CHROMA_OUT): track 4.47 -> 18.3 mm, vias 0 -> 1
- net Net-(IC13-AUDIO_IN): track 41.7 -> 30.2 mm
- net /~{YS}: track 85.9 -> 97.1 mm
- net Net-(IC13-Y_IN): track 23.8 -> 31.9 mm
- net Net-(C28-Pad2): track 11.9 -> 19.8 mm
- net Net-(IC13-R_OUT): track 112.5 -> 106.0 mm
- net Net-(IC13-XO_OUT): track 0.00 -> 5.49 mm, vias 0 -> 1
- net Net-(IC13-AUDIO_OUT): track 108.4 -> 113.6 mm
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Other:
- board text added: "1"
- board text added: "13"
- board text added: "6264 SRAM"
- board text added: "65256 PSRAM"
- board text added: "A1"
- board text added: "A32"
- board text added: "B1"
- board text added: "B32"
- board text added: "CXA1034"
- board text added: "MB3514"
- board text added: "V6.8"
- board text removed: "2413"
- board text removed: "SEGS"
