File: MegaDrive.kicad_sch (KiCad schematic)
At the start: 291 parts, among them J1 Video, J10 Conn_01x04_Pin, J11 Conn_01x02_Pin, J110 Conn_01x04_Pin, J111 Conn_01x02_Socket, J2 Floppy, J3 Cartridge, J4 EXT, J5 Player1, J6 Player2, J7 Jack-DC, J8 AudioJack3, J9 Conn_01x02_Pin, J99 Conn_01x02_Pin, SW1 SW_SPDT, SW2 SW_Push, U1 HD68HC000P8, U10 M5M4C264L, U11 YM2612, U12 CXA1034P, U14 LM358, U15 L7805, U17 L7805, U2 uPD42832C-15, U3 uPD42832C-15, U4 315-5402, U6 Z80CPU, U7 uPD4364, U8 312-5313A, U9 M5M4C264L

Commit message: Add files via upload
Parts:
- added C125: 100pF, Capacitor_SMD:C_0805_2012Metric, symbol MD1_VA6.8:C
- C1, C111, C13, C23, C24, C30, C31, C32, C38, C4, C40, C41, C42, C43, C44, C49, C5, C50, C51, C52, C53, C55, C57, C58, C59, C60, C61, C62, C63, C64, C65, C66, C68, C71, C72, C74, C79, C86, CP112: symbol Device:C_Polarized -> MD1_VA6.8:C_Polarized
- C10, C102, C103, C105, C106, C107, C108, C109, C11, C110, C112, C113, C114, C115, C116, C117, C118, C119, C120, C121, C122, C14, C15, C16, C17, C18, C19, C2, C20, C21, C22, C25, C26, C27, C28, C29, C3, C33, C34, C35, C37, C39, C45, C46, C47, C48, C6, C69, C7, C73, C75, C77, C78, C8, C80, C81, C82, C83, C85, C87, C88, C89, C9, C90, C91, C92, C93, C94, C96: symbol Device:C -> MD1_VA6.8:C
- C95: symbol Device:C -> MD1_VA6.8:C; now not fitted
- CN1: renamed from J1; symbol Connector:DIN-8 -> MD1_VA6.8:DIN-8
- CN10: renamed from J10; symbol Connector:Conn_01x04_Pin -> MD1_VA6.8:Conn_01x04_Pin
- CN11: renamed from J11; symbol Connector:Conn_01x02_Pin -> MD1_VA6.8:Conn_01x02_Pin
- CN110: renamed from J110; symbol Connector:Conn_01x04_Pin -> MD1_VA6.8:Conn_01x04_Pin
- CN111: renamed from J111; symbol Connector:Conn_01x02_Socket -> MD1_VA6.8:Conn_01x02_Socket
- CN2: renamed from J2; symbol Connector_Generic:Conn_02x30_Row_Letter_First -> MD1_VA6.8:Conn_02x30_Row_Letter_First
- CN3: renamed from J3; symbol Connector_Generic:Conn_02x32_Row_Letter_First -> MD1_VA6.8:Conn_02x32_Row_Letter_First
- CN4: renamed from J4; symbol Connector:DE9_Socket -> MD1_VA6.8:DE9_Socket
- CN5: renamed from J5; symbol Connector:DE9_Pins -> MD1_VA6.8:DE9_Pins
- CN6: renamed from J6; symbol Connector:DE9_Pins -> MD1_VA6.8:DE9_Pins
- CN7: renamed from J7; symbol Connector:Jack-DC -> MD1_VA6.8:Jack-DC
- CN8: renamed from J8; symbol Connector_Audio:AudioJack3 -> MD1_VA6.8:AudioJack3
- CN9: renamed from J9; symbol Connector:Conn_01x02_Pin -> MD1_VA6.8:Conn_01x02_Pin
- CN99: renamed from J99; symbol Connector:Conn_01x02_Pin -> MD1_VA6.8:Conn_01x02_Pin
- D1, D2, D3: symbol Device:D -> MD1_VA6.8:D
- EM11, EM12, EM13, EM16, EM21, EM22, EM23, EM24, EM25, EM26, EM27, EM28, EM31, EM32, EM33, EM34, EM35, EM36, EM37, EM38, EM4, EM5, EM7, EM8: symbol Device:C_Feedthrough -> MD1_VA6.8:C_Feedthrough
- FB1, FB10, FB11, FB12, FB13, FB14, FB15, FB2, FB3, FB4, FB5, FB6, FB7, FB8, FB9: symbol Device:FerriteBead -> MD1_VA6.8:FerriteBead
- FID1, FID2, FID3, FID4, FID5, FID6: symbol Mechanical:Fiducial -> MD1_VA6.8:Fiducial
- H1, H10, H11, H12, H13, H14, H15, H2, H3, H4, H5, H6, H7, H8, H9: symbol Mechanical:MountingHole -> MD1_VA6.8:MountingHole
- IC1: renamed from U1; value HD68HC000P8 -> 68000P; symbol CPU_NXP_68000:MC68000P -> MD1_VA6.8:MC68000P
- IC10: renamed from U10; symbol SEGA:M5M4C264L -> MD1_VA6.8:M5M4C264L
- IC11: renamed from U11; symbol ym2612:YM2612 -> MD1_VA6.8:YM2612
- IC12: renamed from U12; symbol SEGA:CXA1034P -> MD1_VA6.8:CXA1034P
- IC13: renamed from U13; value ~ -> MB3514; footprint Package_DIP:DIP-24_W10.16mm -> MegaDrive:SOIC-24_CXA; symbol SEGA:CXA1145P/M -> MD1_VA6.8:CXA1145P/M
- IC14: renamed from U14; symbol Amplifier_Operational:LM358 -> MD1_VA6.8:LM358
- IC15: renamed from U15; symbol Regulator_Linear:L7805 -> MD1_VA6.8:L7805
- IC17: renamed from U17; symbol Regulator_Linear:L7805 -> MD1_VA6.8:L7805
- IC2: renamed from U2; symbol Memory_RAM:CY62256-70PC -> MD1_VA6.8:CY62256-70PC
- IC3: renamed from U3; symbol Memory_RAM:CY62256-70PC -> MD1_VA6.8:CY62256-70PC
- IC4: renamed from U4; value 315-5402 -> 315-5433; symbol SEGA:315-5402 -> MD1_VA6.8:315-5402
- IC6: renamed from U6; symbol CPU:Z80CPU -> MD1_VA6.8:Z80CPU
- IC7: renamed from U7; symbol SEGA:uPD4364 -> MD1_VA6.8:uPD4364
- IC8: renamed from U8; value 312-5313A -> 315-5313A; symbol SEGA:312-5313A -> MD1_VA6.8:312-5313A
- IC9: renamed from U9; symbol SEGA:M5M4C264L -> MD1_VA6.8:M5M4C264L
- JP1, JP4: symbol Jumper:Jumper_2_Open -> MD1_VA6.8:Jumper_2_Open
- JP2, JP3: symbol Jumper:Jumper_2_Bridged -> MD1_VA6.8:Jumper_2_Bridged
- JP5, JP6, JP7: symbol Connector:Conn_01x01_Pin -> MD1_VA6.8:Conn_01x01_Pin
- L2, L3, L5, L6, L7: symbol Device:L -> MD1_VA6.8:L
- NT101: symbol Device:NetTie_2 -> MD1_VA6.8:NetTie_2
- OSC1: symbol Oscillator:VTCXO-14 -> MD1_VA6.8:VTCXO-14
- R1, R10, R11, R12, R14, R15, R16, R17, R18, R19, R20, R21, R22, R23, R24, R25, R26, R29, R3, R30, R31, R32, R33, R34, R35, R36, R37, R38, R39, R4, R40, R41, R42, R43, R49, R5, R50, R51, R52, R53, R54, R55, R56, R57, R58, R59, R6, R64, R65, R66, R67, R68, R69, R7, R70, R71, R72, R73, R74, R77, R78, R79, R8, R80, R81, R82, R83, R84, R85, R9: symbol Device:R -> MD1_VA6.8:R
- R27: value 1.2k -> 560; symbol Device:R -> MD1_VA6.8:R
- R28: value 1.2k -> 3.3k; symbol Device:R -> MD1_VA6.8:R
- RF1: symbol SEGA:RFmod -> MD1_VA6.8:RFmod
- SW1: symbol Switch:SW_SPDT -> MD1_VA6.8:SW_SPDT
- SW2: symbol Switch:SW_Push -> MD1_VA6.8:SW_Push
- VR1: renamed from RV1; symbol Device:R_Potentiometer -> MD1_VA6.8:R_Potentiometer
Connections:
- net GND: now also C125.2
- net at IC13.5 (XO_OUT): now also C125.1
- no-connect marks 34 -> 33
